Commit message: Fixed omnidirectional wheel model

File: src/urdf/arceus_description.urdf (robot description, URDF)
Before this commit: robot arceus, 3 links, 2 joints
Joints:
- joint base_joint: origin xyz=0.0 0.0 ${-(wheel_radius+base_width/2)-0.005} rpy=0 0 0 -> xyz=0.0 0.0 ${-(wheel_radius+base_width/2)-0.008} rpy=0 0 0

Commit message: Added laser filter and changed some variable names

File: src/urdf/arceus_description.urdf (robot description, URDF)
Before this commit: robot arceus, 3 links, 2 joints
Links:
- removed link lidar_link
- added link laser_frame, mass 0.125; collision box size=0.0555 0.0555 0.051; visual box size=0.0555 0.0555 0.051
Joints:
- removed joint lidar_joint
- added joint laser_joint: type fixed, parent base_link, child laser_frame, origin xyz=0 0 ${(base_width/2)+0.0255} rpy=0 0 ${4*pi/3}

Commit message: Fixed motor delay and mapping issues

File: src/urdf/arceus_description.urdf (robot description, URDF)
Before this commit: robot arceus, 3 links, 2 joints
Joints:
- joint laser_joint: origin xyz=0 0 ${(base_width/2)+0.0255} rpy=0 0 ${4*pi/3} -> xyz=0 0 ${(base_width/2)+0.0255} rpy=0 0 0
